Commit message: Add files via upload

File: roborecipe2_description/urdf/roborecipe2.urdf (robot description, URDF)
Before this commit: robot roborecipe1, 36 links, 35 joints
Links:
- link c_chest_dec1: mass 0.000000 -> 0.086483
- link r_ankle: mass 0.000035 -> 0.058000
- link r_arm_lower: mass 0.000049 -> 0.030000
- link r_arm_upper: mass 0.000072 -> 0.098000
- link r_elbow: mass 0.000027 -> 0.044000
- link r_foot_large: mass 0.000064 -> 0.045000
- link r_hipjoint_lower: mass 0.000046 -> 0.058000
- link r_hipjoint_upper: mass 0.000011 -> 0.011500
- link r_leg_lower: mass 0.000022 -> 0.061000
- link r_leg_upper: mass 0.000057 -> 0.091000
- link r_shoulder: mass 0.000020 -> 0.014000
Joints:
- joint base_link_to_c_waist: axis 1 0 0 -> (none); limit lower=-3.14159 upper=3.14159 effort=0 velocity=0 -> (none)
- joint c_chest_to_c_head: origin xyz=0.01145 1e-06 0.0624 rpy=0.0 0.0 0.0 -> xyz=0.01145 -0.0 0.0624 rpy=0.0 0.0 0.0
- joint c_chest_to_l_shoulder: origin xyz=0.01147 0.048948 0.0454 rpy=0.0 0.0 0.0 -> xyz=0.01145 0.04885 0.0454 rpy=0.0 0.0 0.0
- joint c_chest_to_r_shoulder: origin xyz=0.01147 -0.048948 0.0454 rpy=0.0 0.0 0.0 -> xyz=0.01145 -0.04885 0.0454 rpy=0.0 0.0 0.0
